Commit message: fix obstacle recognition due to lidar recognizing parts of robot

File: simulations/ros_lidar_simulation/src/track_spray_robot/urdf/track_spray_robot.urdf (robot description, URDF)
Before this commit: robot track_spray_robot, 7 links, 6 joints
Links:
- link lidar_link: geometry visual cylinder length=0.1 radius=0.05
